File: encoder v2.0/encoder v2.0.sch (KiCad schematic (older format))
At the start: 15 parts, among them J1 Conn_01x02, J2 Conn_01x03, J3 Conn_01x05, J4 Conn_01x01, J5 Conn_01x05, U1 74LS14

Commit message: finalizando el ruteo
Parts:
- H1, H2, H3, H4: footprint MountingHole:MountingHole_4mm_Pad_Via -> MountingHole:MountingHole_3mm_Pad
Changed lines of the file:
@@
 F 0 "H1" H 9700 5196 50  0000 L CNN
 F 1 "MountingHole" H 9700 5105 50  0000 L CNN
-F 2 "MountingHole:MountingHole_4mm_Pad_Via" H 9600 5150 50  0001 C CNN
+F 2 "MountingHole:MountingHole_3mm_Pad" H 9600 5150 50  0001 C CNN
 F 3 "~" H 9600 5150 50  0001 C CNN
 	1    9600 5150
@@
 F 0 "H3" H 10500 5196 50  0000 L CNN
 F 1 "MountingHole" H 10500 5105 50  0000 L CNN
-F 2 "MountingHole:MountingHole_4mm_Pad_Via" H 10400 5150 50  0001 C CNN
+F 2 "MountingHole:MountingHole_3mm_Pad" H 10400 5150 50  0001 C CNN
 F 3 "~" H 10400 5150 50  0001 C CNN
 	1    10400 5150
@@
 F 0 "H2" H 9700 5496 50  0000 L CNN
 F 1 "MountingHole" H 9700 5405 50  0000 L CNN
-F 2 "MountingHole:MountingHole_4mm_Pad_Via" H 9600 5450 50  0001 C CNN
+F 2 "MountingHole:MountingHole_3mm_Pad" H 9600 5450 50  0001 C CNN
 F 3 "~" H 9600 5450 50  0001 C CNN
 	1    9600 5450
@@
 F 0 "H4" H 10500 5496 50  0000 L CNN
 F 1 "MountingHole" H 10500 5405 50  0000 L CNN
-F 2 "MountingHole:MountingHole_4mm_Pad_Via" H 10400 5450 50  0001 C CNN
+F 2 "MountingHole:MountingHole_3mm_Pad" H 10400 5450 50  0001 C CNN
 F 3 "~" H 10400 5450 50  0001 C CNN
 	1    10400 5450

Commit message: Ruteo finalizado y realizar una verificación
Parts:
- added J6: Conn_01x01, Connector_PinHeader_2.54mm:PinHeader_1x01_P2.54mm_Vertical, symbol Connector_Generic:Conn_01x01
- added JP1: Jumper_3_Open, Connector_PinHeader_2.54mm:PinHeader_1x03_P2.54mm_Vertical, symbol Jumper:Jumper_3_Open
- J1: footprint TerminalBlock_Phoenix:TerminalBlock_Phoenix_MKDS-1,5-2-5.08_1x02_P5.08mm_Horizontal -> Terminal Degson:dg126
Connections:
- net at C2.1, R2.2, U1.1: now also JP1.1 (A); no longer J2.3 (Pin_3)
- new net: J6.1 (Pin_1), JP1.3 (B)
- new net: J2.3 (Pin_3), JP1.2 (C)
Changed lines of the file:
@@
 F 0 "J1" H 818 1025 50  0000 C CNN
 F 1 "Conn_01x02" H 818 1116 50  0000 C CNN
-F 2 "TerminalBlock_Phoenix:TerminalBlock_Phoenix_MKDS-1,5-2-5.08_1x02_P5.08mm_Horizontal" H 900 1350 50  0001 C CNN
+F 2 "Terminal Degson:dg126" H 900 1350 50  0001 C CNN
 F 3 "~" H 900 1350 50  0001 C CNN
 	1    900  1350
@@
 Wire Wire Line
 	4100 1500 4100 1550
-Wire Wire Line
-	3600 1600 3600 2100
-Wire Wire Line
-	3600 2100 4650 2100
-Wire Wire Line
-	4650 2100 4650 1600
-Wire Wire Line
-	4650 1600 5200 1600
 Wire Notes Line
 	3450 1150 3400 1000
@@
 Wire Wire Line
 	3600 1500 4100 1500
+$Comp
+L Connector_Generic:Conn_01x01 J6
+U 1 1 5ED722D6
+P 4150 2400
+F 0 "J6" H 4230 2442 50  0000 L CNN
+F 1 "Conn_01x01" H 4230 2351 50  0000 L CNN
+F 2 "Connector_PinHeader_2.54mm:PinHeader_1x01_P2.54mm_Vertical" H 4150 2400 50  0001 C CNN
+F 3 "~" H 4150 2400 50  0001 C CNN
+	1    4150 2400
+	1    0    0    -1
+$EndComp
+$Comp
+L Jumper:Jumper_3_Open JP1
+U 1 1 5ED73947
+P 3850 2150
+F 0 "JP1" V 3804 2237 50  0000 L CNN
+F 1 "Jumper_3_Open" V 3895 2237 50  0000 L CNN
+F 2 "Connector_PinHeader_2.54mm:PinHeader_1x03_P2.54mm_Vertical" H 3850 2150 50  0001 C CNN
+F 3 "~" H 3850 2150 50  0001 C CNN
+	1    3850 2150
+	0    1    1    0
+$EndComp
+Wire Wire Line
+	3600 1600 3600 2150
+Wire Wire Line
+	3600 2150 3700 2150
+Wire Wire Line
+	3850 1900 4450 1900
+Wire Wire Line
+	4450 1900 4450 1600
+Wire Wire Line
+	4450 1600 5200 1600
+Wire Wire Line
+	3850 2400 3950 2400
 $EndSCHEMATC
